File: pcb/pin-check.sch (KiCad schematic (older format))
At the start: 39 parts, among them P1 USB_C_Receptacle_USB2.0, SW1 SW_Push, SW2 SW_Push, SW3 SW_Push, SW4 SW_Push, SW5 SW_Push, SW6 SW_Push, SW7 Reset, SW8 Boot, U1 ATmega328P-PU, Y1 16MHz

Commit message: still a wip, uploading bom
Parts:
- added H12, H13, H14, H15, H16, H17: Pad, Connector_PinSocket_2.00mm:PinSocket_1x01_P2.00mm_Vertical, symbol Mechanical:MountingHole_Pad
- renumbered H4 to H10, H5 to H11, H6 to H2, H7 to H3, H8 to H4, H9 to H5, H10 to H6, H11 to H7, H2 to H8, H3 to H9
Connections:
- net D6: now reaches U1.12 (PD6)
- net D6: now also H16.1
- net D7: now reaches U1.13 (PD7)
- net D7: now also H17.1
- net D0: now reaches U1.2 (PD0)
- net D0: now also H13.1
- net C5: now reaches U1.28 (PC5)
- net C5: now also H12.1
- net D1: now reaches U1.3 (PD1)
- net D1: now also H14.1
- net D4: now reaches U1.6 (PD4)
- net D4: now also H15.1
- net Row1 renamed B1
- net Row2 renamed B2
- net Row3 renamed B3
- net Row4 renamed B4
- no-connect marks 9 -> 3
Other:
- moved on the sheet: H1, H10, H11, H2, H3, H4, H5, H6, H7, H8, H9

Commit message: a bunch of changes, update bom, new render
Parts:
- added C3: 4.7u, Capacitor_THT:C_Radial_D4.0mm_H7.0mm_P1.50mm, symbol Device:C
- added C4, C5: 0.1u, Capacitor_THT:C_Rect_L4.0mm_W2.5mm_P2.50mm, symbol Device:C
- added D9: LED, LED_THT:LED_D3.0mm, symbol Device:LED
- added H18, H19, H20, H21: MountingHole, MountingHole:MountingHole_2.2mm_M2, symbol Mechanical:MountingHole
- added J1: AVR-ISP-6, Connector_PinHeader_2.54mm:PinHeader_2x03_P2.54mm_Horizontal, symbol Connector:AVR-ISP-6
- added R7: 1.5k, Resistor_THT:R_Axial_DIN0204_L3.6mm_D1.6mm_P7.62mm_Horizontal, symbol Device:R
- C1, C2: footprint Capacitor_THT:C_Radial_D6.3mm_H5.0mm_P2.50mm -> Capacitor_THT:C_Rect_L4.0mm_W2.5mm_P2.50mm
- D1, D2, D3, D4, D5, D6, D7, D8: footprint Diode_THT:D_DO-35_SOD27_P7.62mm_Horizontal -> pin-check:D_DO-35_SOD27_P5.08mm_Horizontal
- F1: footprint Fuse:Fuse_Bourns_MF-RG300 -> Fuse:Fuse_Littelfuse_395Series
- H1, H10, H11, H12, H13, H14, H15, H16, H17, H2, H3, H4, H5, H6, H7, H8, H9: footprint Connector_PinSocket_2.00mm:PinSocket_1x01_P2.00mm_Vertical -> Connector_Wire:SolderWire-0.5sqmm_1x01_D0.9mm_OD2.1mm
- R1, R2, R3, R4, R5, R6: footprint Resistor_THT:R_Axial_DIN0207_L6.3mm_D2.5mm_P10.16mm_Horizontal -> Resistor_THT:R_Axial_DIN0204_L3.6mm_D1.6mm_P7.62mm_Horizontal
Connections:
- net +5V: now also C3.2, C4.2, C5.2, D9.2 (A), J1.2 (VCC)
- net B3: now also J1.4 (MOSI)
- net B4: now also J1.1 (MISO)
- net Col0: now also J1.3 (SCK)
- net GND: now also C3.1, C4.1, C5.1, J1.6 (GND), R7.2
- net Reset: now also J1.5 (~RST)
- new net: D9.1 (K), R7.1
Other:
- note added: "Boot and Reset Switches"
- note added: "Decoupling Capacitors"
- note added: "Keyswitches and Diodes"
- note added: "Microcontroller, Crystal, and ISP Headers"
- note added: "Mounting Holes"
- note added: "Power LED"
- note added: "Solder Pads For Additional Rows and Columns"
- note added: "USB Port"
- moved on the sheet: C1, C2, D1, D2, D3, D4, D5, D6, D7, D8, F1, H1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

Commit message: update images and move usb port down
Parts:
- P1: footprint Connector_USB:USB_C_Receptacle_GCT_USB4085 -> pin-check:USB_C_GCT_USB4085
Other:
- moved on the sheet: H18, H19, H20, H21
Changed lines of the file:
@@
 Title "pin-check"
 Date ""
-Rev "v0.0.1"
+Rev "v0.0.2"
 Comp ""
 Comment1 ""
@@
 F 0 "P1" H 7650 2350 50  0000 C CNN
 F 1 "USB_C_Receptacle_USB2.0" H 7200 2250 50  0000 C CNN
-F 2 "Connector_USB:USB_C_Receptacle_GCT_USB4085" H 8300 2250 50  0001 C CNN
+F 2 "pin-check:USB_C_GCT_USB4085" H 8300 2250 50  0001 C CNN
 F 3 "https://www.usb.org/sites/default/files/documents/usb_type-c.zip" H 8300 2250 50  0001 C CNN
 	1    8150 2250
@@
 L Mechanical:MountingHole H18
 U 1 1 5F14FC44
-P 8450 6100
-F 0 "H18" H 8550 6146 50  0000 L CNN
-F 1 "MountingHole" H 8550 6055 50  0000 L CNN
-F 2 "MountingHole:MountingHole_2.2mm_M2" H 8450 6100 50  0001 C CNN
-F 3 "~" H 8450 6100 50  0001 C CNN
-	1    8450 6100
+P 8000 6050
+F 0 "H18" H 8100 6096 50  0000 L CNN
+F 1 "MountingHole" H 8100 6005 50  0000 L CNN
+F 2 "MountingHole:MountingHole_2.2mm_M2" H 8000 6050 50  0001 C CNN
+F 3 "~" H 8000 6050 50  0001 C CNN
+	1    8000 6050
 	1    0    0    -1
 $EndComp
@@
 L Mechanical:MountingHole H20
 U 1 1 5F150145
-P 9200 6100
-F 0 "H20" H 9300 6146 50  0000 L CNN
-F 1 "MountingHole" H 9300 6055 50  0000 L CNN
-F 2 "MountingHole:MountingHole_2.2mm_M2" H 9200 6100 50  0001 C CNN
-F 3 "~" H 9200 6100 50  0001 C CNN
-	1    9200 6100
+P 8750 6050
+F 0 "H20" H 8850 6096 50  0000 L CNN
+F 1 "MountingHole" H 8850 6005 50  0000 L CNN
+F 2 "MountingHole:MountingHole_2.2mm_M2" H 8750 6050 50  0001 C CNN
+F 3 "~" H 8750 6050 50  0001 C CNN
+	1    8750 6050
 	1    0    0    -1
 $EndComp
@@
 L Mechanical:MountingHole H19
 U 1 1 5F15037C
-P 8450 6300
-F 0 "H19" H 8550 6346 50  0000 L CNN
-F 1 "MountingHole" H 8550 6255 50  0000 L CNN
-F 2 "MountingHole:MountingHole_2.2mm_M2" H 8450 6300 50  0001 C CNN
-F 3 "~" H 8450 6300 50  0001 C CNN
-	1    8450 6300
+P 8000 6250
+F 0 "H19" H 8100 6296 50  0000 L CNN
+F 1 "MountingHole" H 8100 6205 50  0000 L CNN
+F 2 "MountingHole:MountingHole_2.2mm_M2" H 8000 6250 50  0001 C CNN
+F 3 "~" H 8000 6250 50  0001 C CNN
+	1    8000 6250
 	1    0    0    -1
 $EndComp
@@
 L Mechanical:MountingHole H21
 U 1 1 5F151956
-P 9200 6300
-F 0 "H21" H 9300 6346 50  0000 L CNN
-F 1 "MountingHole" H 9300 6255 50  0000 L CNN
-F 2 "MountingHole:MountingHole_2.2mm_M2" H 9200 6300 50  0001 C CNN
-F 3 "~" H 9200 6300 50  0001 C CNN
-	1    9200 6300
-	1    0    0    -1
-$EndComp
-Text Notes 8750 5950 0    63   ~ 0
+P 8750 6250
+F 0 "H21" H 8850 6296 50  0000 L CNN
+F 1 "MountingHole" H 8850 6205 50  0000 L CNN
+F 2 "MountingHole:MountingHole_2.2mm_M2" H 8750 6250 50  0001 C CNN
+F 3 "~" H 8750 6250 50  0001 C CNN
+	1    8750 6250
+	1    0    0    -1
+$EndComp
+Text Notes 8300 5900 0    63   ~ 0
 Mounting Holes
 $Comp
