File: pcb/pin-check.sch (KiCad schematic (older format))
At the start: 52 parts, among them J1 AVR-ISP-6, J2 SJ-43514, P1 USB_C_Receptacle_USB2.0, SW1 MX-NoLED, SW2 MX-NoLED, SW3 MX-NoLED, SW4 MX-NoLED, SW7 Reset, SW8 Boot, U1 ATmega328P-PU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

Commit message: probably not
Parts:
- removed U1: ATmega328P-PU, Package_DIP:DIP-28_W7.62mm, symbol MCU_Microchip_ATmega:ATmega328P-PU
- added U1: ATmega32A-PU, Package_DIP:DIP-40_W15.24mm, symbol MCU_Microchip_ATmega:ATmega32A-PU
Connections:
- net labels added: C0, C1
- no-connect marks 3 -> 2
Other:
- moved on the sheet: C1, C2, J1, Y1

Commit message: asdf
Parts:
- added H18, H19, H20, H21, H22, H23, H24: Pad, Connector_Wire:SolderWire-0.5sqmm_1x01_D0.9mm_OD2.1mm, symbol Mechanical:MountingHole_Pad
- renumbered H18 to H25, H19 to H26, H20 to H27, H21 to H28
Connections:
- net labels added: A0, A1, A2, A3, B0, C2, C6, C7, D5, SCL, SDA
- net labels removed: C0, C1, D4, D6
- no-connect marks 2 -> 3
Other:
- moved on the sheet: C3, C4, C5, D1, D2, D3, D4, H14, H15, H16, H17, H25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
