File: pcb/pin-check.kicad_pcb (KiCad board)
At the start: 2 copper layers, 114.3 x 44.2 mm, 56 parts, among them J1 AVR-ISP-6, P1 USB_C_Receptacle_USB2.0, SW1 SW_Push, SW2 SW_Push, SW3 SW_Push, SW4 SW_Push, SW5 SW_Push, SW6 SW_Push, SW7 Reset, SW8 Boot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

Commit message: schematic pdf
Parts:
- moved C2 0.51 mm to (60.5, 39.9)
- moved C3 0.51 mm to (87.1, 37.8)
- moved C4 0.51 mm to (81.5, 37.3)
- moved Y1 0.51 mm to (66.5, 38.7)
- moved C1 0.43 mm to (77.7, 39.9)
Routing:
- net +5V: track 125.3 -> 124.2 mm
Changed lines of the file:
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@@
     (thickness 1.6)
     (drawings 7)
-    (tracks 328)
+    (tracks 331)
     (zones 0)
     (modules 56)
@@
   )
   (module Capacitor_THT:C_Radial_D4.0mm_H7.0mm_P1.50mm (layer F.Cu)
-    (at 87.63 37.846 270)
+    (at 87.122 37.846 270)
     (descr "C, Radial series, Radial, pin pitch=1.50mm, diameter=4mm, height=7mm, Non-Polar Electrolytic Capacitor")
     (tags "C Radial series Radial pin pitch 1.50mm diameter 4mm height 7mm Non-Polar Electrolytic Capacitor")
@@
   )
   (module Crystal:Crystal_HC49-4H_Vertical (layer F.Cu)
-    (at 67.056 38.735)
+    (at 66.548 38.735)
     (descr "Crystal THT HC-49-4H http://5hertz.com/pdfs/04404_D.pdf")
     (tags "THT crystalHC-49-4H")
@@
   )
   (module Capacitor_THT:C_Rect_L4.0mm_W2.5mm_P2.50mm (layer F.Cu)
-    (at 82.042 37.338 270)
+    (at 81.534 37.338 270)
     (descr "C, Rect series, Radial, pin pitch=2.50mm, , length*width=4*2.5mm^2, Capacitor")
     (tags "C Rect series Radial pin pitch 2.50mm  length 4mm width 2.5mm Capacitor")
@@
   )
   (module Capacitor_THT:C_Rect_L4.0mm_W2.5mm_P2.50mm (layer F.Cu)
-    (at 60.96 39.878 90)
+    (at 60.452 39.878 90)
     (descr "C, Rect series, Radial, pin pitch=2.50mm, , length*width=4*2.5mm^2, Capacitor")
     (tags "C Rect series Radial pin pitch 2.50mm  length 4mm width 2.5mm Capacitor")
@@
   )
   (module Capacitor_THT:C_Rect_L4.0mm_W2.5mm_P2.50mm (layer F.Cu)
-    (at 78.1558 39.878 90)
+    (at 77.724 39.878 90)
     (descr "C, Rect series, Radial, pin pitch=2.50mm, , length*width=4*2.5mm^2, Capacitor")
     (tags "C Rect series Radial pin pitch 2.50mm  length 4mm width 2.5mm Capacitor")
@@
   (gr_line (start 44.45 57.023) (end 44.45 77.724) (layer Edge.Cuts) (width 0.05))
   (gr_line (start 158.75 77.724) (end 44.45 77.724) (layer Edge.Cuts) (width 0.05))
-  (segment (start 76.7988 38.735) (end 78.1558 37.378) (width 0.3) (layer F.Cu) (net 1) (status 20))
-  (segment (start 71.936 38.735) (end 76.7988 38.735) (width 0.3) (layer F.Cu) (net 1) (status 10))
-  (segment (start 70.1548 40.5162) (end 71.936 38.735) (width 0.3) (layer B.Cu) (net 1) (status 20))
-  (segment (start 70.1548 44.196) (end 70.1548 40.5162) (width 0.3) (layer B.Cu) (net 1) (status 10))
+  (segment (start 76.367 38.735) (end 77.724 37.378) (width 0.3) (layer F.Cu) (net 1))
+  (segment (start 71.428 38.735) (end 76.367 38.735) (width 0.3) (layer F.Cu) (net 1))
+  (segment (start 70.1548 40.0082) (end 71.428 38.735) (width 0.3) (layer B.Cu) (net 1))
+  (segment (start 70.1548 44.196) (end 70.1548 40.0082) (width 0.3) (layer B.Cu) (net 1))
   (segment (start 121.262 36.14) (end 127.762 36.14) (width 0.3) (layer B.Cu) (net 2) (status 30))
   (segment (start 135.994 36.14) (end 142.494 36.14) (width 0.3) (layer B.Cu) (net 2) (status 30))
   (segment (start 135.994 36.14) (end 127.762 36.14) (width 0.3) (layer F.Cu) (net 2) (status 30))
-  (segment (start 62.317 38.735) (end 60.96 37.378) (width 0.3) (layer F.Cu) (net 3) (status 20))
-  (segment (start 67.056 38.735) (end 62.317 38.735) (width 0.3) (layer F.Cu) (net 3) (status 10))
-  (segment (start 67.6148 39.2938) (end 67.056 38.735) (width 0.3) (layer B.Cu) (net 3) (status 20))
-  (segment (start 67.6148 44.196) (end 67.6148 39.2938) (width 0.3) (layer B.Cu) (net 3) (status 10))
-  (segment (start 75.2348 44.196) (end 75.2348 42.3672) (width 0.6) (layer B.Cu) (net 4) (status 10))
-  (segment (start 75.2348 42.3672) (end 76.2 41.402) (width 0.6) (layer B.Cu) (net 4))
-  (segment (start 80.478 41.402) (end 82.042 39.838) (width 0.6) (layer B.Cu) (net 4) (status 20))
-  (segment (start 76.2 41.402) (end 80.478 41.402) (width 0.6) (layer B.Cu) (net 4))
-  (segment (start 87.138 39.838) (end 87.63 39.346) (width 0.6) (layer F.Cu) (net 4) (status 20))
-  (segment (start 82.042 39.838) (end 87.138 39.838) (width 0.6) (layer F.Cu) (net 4) (status 10))
+  (segment (start 67.6148 39.8018) (end 66.548 38.735) (width 0.3) (layer B.Cu) (net 3))
+  (segment (start 67.6148 44.196) (end 67.6148 39.8018) (width 0.3) (layer B.Cu) (net 3))
+  (segment (start 66.548 38.735) (end 61.809 38.735) (width 0.3) (layer F.Cu) (net 3))
+  (segment (start 61.809 38.735) (end 60.452 37.378) (width 0.3) (layer F.Cu) (net 3))
   (segment (start 75.2348 46.736) (end 70.1548 51.816) (width 0.6) (layer B.Cu) (net 4) (status 20))
   (segment (start 75.2348 44.196) (end 75.2348 46.736) (width 0.6) (layer B.Cu) (net 4) (status 10))
@@
   (segment (start 70.104 51.8668) (end 70.1548 51.816) (width 0.6) (layer F.Cu) (net 4) (status 30))
   (segment (start 70.104 53.7572) (end 70.104 51.8668) (width 0.6) (layer F.Cu) (net 4) (status 20))
-  (segment (start 88.039122 39.346) (end 87.63 39.346) (width 0.6) (layer B.Cu) (net 4) (status 30))
-  (segment (start 94.549523 45.856401) (end 88.039122 39.346) (width 0.6) (layer B.Cu) (net 4) (status 20))
   (segment (start 100.701599 45.856401) (end 94.549523 45.856401) (width 0.6) (layer B.Cu) (net 4))
   (segment (start 101.854 44.704) (end 100.701599 45.856401) (width 0.6) (layer B.Cu) (net 4) (status 10))
@@
   (segment (start 131.572 39.389378) (end 131.572 34.798) (width 0.6) (layer B.Cu) (net 4) (status 20))
   (segment (start 128.152689 42.808689) (end 131.572 39.389378) (width 0.6) (layer B.Cu) (net 4))
+  (segment (start 91.093523 42.400401) (end 94.549523 45.856401) (width 0.6) (layer B.Cu) (net 4))
+  (segment (start 90.176401 42.400401) (end 91.093523 42.400401) (width 0.6) (layer B.Cu) (net 4))
+  (segment (start 87.122 39.346) (end 90.176401 42.400401) (width 0.6) (layer B.Cu) (net 4))
+  (segment (start 75.2348 44.196) (end 77.7748 41.656) (width 0.6) (layer B.Cu) (net 4))
+  (segment (start 79.716 41.656) (end 81.534 39.838) (width 0.6) (layer B.Cu) (net 4))
+  (segment (start 77.7748 41.656) (end 79.716 41.656) (width 0.6) (layer B.Cu) (net 4))
+  (segment (start 86.63 39.838) (end 87.122 39.346) (width 0.6) (layer B.Cu) (net 4))
+  (segment (start 81.534 39.838) (end 86.63 39.838) (width 0.6) (layer B.Cu) (net 4))
   (segment (start 123.317 56.007) (end 123.317 49.5935) (width 0.3) (layer F.Cu) (net 5) (status 20))
   (segment (start 120.142 59.182) (end 123.317 56.007) (width 0.3) (layer F.Cu) (net 5))
@@
   (segment (start 104.0756 40.5756) (end 104.0756 40.843) (width 0.3) (layer F.Cu) (net 14) (status 30))
   (segment (start 103.54059 40.04059) (end 104.0756 40.5756) (width 0.3) (layer F.Cu) (net 14) (status 20))
-  (segment (start 104.43301 39.68559) (end 104.0756 40.043) (width 0.3) (layer F.Cu) (net 14))
-  (segment (start 104.0756 40.043) (end 104.0756 40.843) (width 0.3) (layer F.Cu) (net 14) (status 20))
-  (segment (start 106.592258 39.68559) (end 104.43301 39.68559) (width 0.3) (layer F.Cu) (net 14))
-  (segment (start 110.5 43.593332) (end 106.592258 39.68559) (width 0.3) (layer F.Cu) (net 14))
-  (segment (start 110.5 45.974) (end 110.5 43.593332) (width 0.3) (layer F.Cu) (net 14) (status 10))
   (segment (start 104.0756 42.163) (end 104.0806 42.168) (width 0.3) (layer B.Cu) (net 14) (status 30))
-  (segment (start 104.0756 40.843) (end 104.0756 42.163) (width 0.3) (layer B.Cu) (net 14) (status 30))
   (segment (start 99.8256 42.163) (end 99.8306 42.168) (width 0.3) (layer B.Cu) (net 14) (status 30))
   (segment (start 99.8256 40.843) (end 99.8256 42.163) (width 0.3) (layer B.Cu) (net 14) (status 30))
+  (segment (start 104.0806 40.848) (end 104.0756 40.843) (width 0.6) (layer B.Cu) (net 14))
+  (segment (start 104.0806 42.168) (end 104.0806 40.848) (width 0.6) (layer B.Cu) (net 14))
+  (segment (start 106.65439 39.53559) (end 107.95 40.8312) (width 0.6) (layer F.Cu) (net 14))
+  (segment (start 104.28301 39.53559) (end 106.65439 39.53559) (width 0.6) (layer F.Cu) (net 14))
+  (segment (start 104.0756 39.743) (end 104.28301 39.53559) (width 0.6) (layer F.Cu) (net 14))
+  (segment (start 104.0756 40.843) (end 104.0756 39.743) (width 0.6) (layer F.Cu) (net 14))
+  (segment (start 107.95 42.950378) (end 110.5 45.500378) (width 0.6) (layer F.Cu) (net 14))
+  (segment (start 110.5 45.500378) (end 110.5 45.974) (width 0.6) (layer F.Cu) (net 14))
+  (segment (start 107.95 40.8312) (end 107.95 42.950378) (width 0.6) (layer F.Cu) (net 14))
   (segment (start 56.5 76.1215) (end 56.515 76.1365) (width 0.3) (layer B.Cu) (net 15) (status 30))
   (segment (start 56.5 61.5) (end 56.5 76.1215) (width 0.3) (layer B.Cu) (net 15) (status 30))

Commit message: smaller!
Parts:
- removed D5, D6: 1N4148, pin-check:D_DO-35_SOD27_P5.08mm_Horizontal
- removed D9: LED, LED_THT:LED_D3.0mm
- removed the G*** at (115.8, 38.6)
- removed R7: 1.5k, Resistor_THT:R_Axial_DIN0204_L3.6mm_D1.6mm_P7.62mm_Horizontal
- removed SW5, SW6: SW_Push, Button_Switch_Keyboard:SW_Cherry_MX_1.00u_PCB
- added G***: LOGO, pin-check:pin-check-pattern, F.Cu at (117.3, 55.5)
- added G***: LOGO, pin-check:pin-check-pattern, F.Cu at (96.6, 55.5)
- D1, D2, D3, D4: moved to B.Cu
- J1: footprint Connector_PinHeader_2.54mm:PinHeader_2x03_P2.54mm_Horizontal -> Connector_PinHeader_2.54mm:PinHeader_2x03_P2.54mm_Vertical
- moved H3 48.4 mm to (120.7, 58.6)
- moved H2 48.4 mm to (101.6, 58.6)
- moved H4 48.4 mm to (139.7, 58.6)
- moved D1 47.9 mm to (83.8, 70.4), turned to 90 degrees
- moved H5 43.3 mm to (156.9, 76.2)
- moved R2 43.0 mm to (138.5, 55.3), turned to 0 degrees
- moved H1 40.2 mm to (84.4, 76.2)
- moved C2 39.6 mm to (99.8, 35.6), turned to 0 degrees
- moved R3 39.0 mm to (137.5, 52.8), turned to 0 degrees
- moved D7 38.6 mm to (130.5, 42.5), turned to 90 degrees
- moved SW2 38.1 mm to (113.7, 61.5)
- moved SW1 38.1 mm to (94.6, 61.5)
- moved SW3 38.1 mm to (132.7, 61.5)
- moved SW4 38.1 mm to (151.8, 61.5)
- moved H18 37.8 mm to (94.0, 36.1)
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Connections:
- H10 pad 1: /B3 -> /D7
- H11 pad 1: /B4 -> /C5
- H12 pad 1: /C5 -> /C4
- H13 pad 1: /D0 -> /C3
- H14 pad 1: /D1 -> /B4
- H15 pad 1: /D4 -> /B3
- H16 pad 1: /D6 -> /B2
- H17 pad 1: /D7 -> /B1
- H6 pad 1: /Col4 -> /D0
- H7 pad 1: /Col5 -> /D1
- H8 pad 1: /B1 -> /D4
- H9 pad 1: /B2 -> /D6
- U1 pad 26: /Col4 -> /C3
- U1 pad 27: /Col5 -> /C4
Routing:
- net /Col5: track 100.1 -> 0.00 mm
- net /Col4: track 80.1 -> 0.00 mm
- net Net-(D1-Pad2): track 82.9 -> 4.44 mm
- net Net-(D2-Pad2): track 65.1 -> 5.70 mm
- net /Col0: track 128.6 -> 81.5 mm, vias 7 -> 2
- net Net-(D3-Pad2): track 47.2 -> 5.73 mm
- net /D7: track 29.4 -> 66.1 mm, vias 1 -> 0
- net +5V: track 124.2 -> 88.1 mm
- net /B1: track 62.1 -> 29.9 mm
- net /D6: track 30.6 -> 62.9 mm, vias 1 -> 0
- net /Reset: track 75.7 -> 46.5 mm, vias 3 -> 1
- net /B2: track 58.4 -> 29.9 mm
- net Net-(P1-PadB5): track 9.89 -> 36.5 mm
- net Net-(D4-Pad2): track 31.3 -> 5.70 mm
- net /C3: track 0.00 -> 24.6 mm
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Other:
- board size 114.3 x 44.2 mm -> 76.2 x 44.2 mm
- board text added: "BOOT"
- board text added: "RESET"
- board text added: "pin-check v0.1.0 by brian"
- board text removed: "pin-check v0.0.2 by brian"

Commit message: I forget
Parts:
- moved C1 0.38 mm to (109.7, 35.9)
- moved C2 0.38 mm to (99.8, 35.9)
Routing:
- net GND: vias 0 -> 2
Changed lines of the file:
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@@
     (thickness 1.6)
     (drawings 9)
-    (tracks 295)
+    (tracks 299)
     (zones 0)
     (modules 51)
@@
     (descr "Fuse, TE5, Littelfuse/Wickmann, No. 460, No560,")
     (tags "Fuse TE5 Littelfuse/Wickmann No. 460 No560 ")
-    (fp_text reference F1 (at 2.4892 0) (layer F.SilkS)
+    (fp_text reference F1 (at 2.4892 -3.0734) (layer F.SilkS)
       (effects (font (size 1 1) (thickness 0.15)))
     )
@@
     (descr "C, Rect series, Radial, pin pitch=2.50mm, , length*width=4*2.5mm^2, Capacitor")
     (tags "C Rect series Radial pin pitch 2.50mm  length 4mm width 2.5mm Capacitor")
-    (fp_text reference C4 (at -2.286 0 90) (layer F.SilkS)
+    (fp_text reference C4 (at -2.032 0 90) (layer F.SilkS)
       (effects (font (size 1 1) (thickness 0.15)))
     )
@@
   )
   (module Capacitor_THT:C_Rect_L4.0mm_W2.5mm_P2.50mm (layer F.Cu)
-    (at 99.822 35.56)
+    (at 99.822 35.941)
     (descr "C, Rect series, Radial, pin pitch=2.50mm, , length*width=4*2.5mm^2, Capacitor")
     (tags "C Rect series Radial pin pitch 2.50mm  length 4mm width 2.5mm Capacitor")
@@
   )
   (module Capacitor_THT:C_Rect_L4.0mm_W2.5mm_P2.50mm (layer F.Cu)
-    (at 109.728 35.56 180)
+    (at 109.728 35.941 180)
     (descr "C, Rect series, Radial, pin pitch=2.50mm, , length*width=4*2.5mm^2, Capacitor")
     (tags "C Rect series Radial pin pitch 2.50mm  length 4mm width 2.5mm Capacitor")
@@
   (segment (start 107.242 40.64) (end 103.124 44.758) (width 0.3) (layer F.Cu) (net 1) (status 30))
   (segment (start 107.242 35.574) (end 107.228 35.56) (width 0.3) (layer F.Cu) (net 1) (status 30))
-  (segment (start 107.242 40.64) (end 107.242 35.574) (width 0.3) (layer F.Cu) (net 1) (status 30))
+  (segment (start 107.242 35.955) (end 107.228 35.941) (width 0.3) (layer F.Cu) (net 1))
+  (segment (start 107.242 40.64) (end 107.242 35.955) (width 0.3) (layer F.Cu) (net 1))
   (segment (start 123.625 42.168) (end 123.625 40.843) (width 0.5) (layer F.Cu) (net 2) (status 30))
   (segment (start 117.675 40.848) (end 117.67 40.843) (width 0.5) (layer F.Cu) (net 2) (status 30))
   (segment (start 117.675 42.168) (end 117.675 40.848) (width 0.5) (layer F.Cu) (net 2) (status 30))
+  (via (at 127 67.691) (size 0.6858) (drill 0.3302) (layers F.Cu B.Cu) (net 2))
+  (via (at 88.9 67.691) (size 0.6858) (drill 0.3302) (layers F.Cu B.Cu) (net 2))
   (segment (start 108.204 55.626) (end 108.204 52.832) (width 0.6) (layer F.Cu) (net 2) (status 30))
   (segment (start 100.584 42.418) (end 102.362 40.64) (width 0.3) (layer F.Cu) (net 3) (status 20))
   (segment (start 100.584 45.212) (end 100.584 42.418) (width 0.3) (layer F.Cu) (net 3) (status 10))
   (segment (start 102.362 35.6) (end 102.322 35.56) (width 0.3) (layer F.Cu) (net 3) (status 30))
-  (segment (start 102.362 40.64) (end 102.362 35.6) (width 0.3) (layer F.Cu) (net 3) (status 30))
+  (segment (start 102.362 35.981) (end 102.322 35.941) (width 0.3) (layer F.Cu) (net 3))
+  (segment (start 102.362 40.64) (end 102.362 35.981) (width 0.3) (layer F.Cu) (net 3))
   (segment (start 111.546 41.87) (end 112.903 41.87) (width 0.6) (layer F.Cu) (net 4) (status 20))
   (segment (start 108.204 45.212) (end 111.546 41.87) (width 0.6) (layer F.Cu) (net 4) (status 10))
@@
   (segment (start 127.09641 43.07041) (end 123.323697 43.07041) (width 0.5) (layer F.Cu) (net 12))
   (via (at 131.45 50.424) (size 0.6858) (drill 0.3302) (layers F.Cu B.Cu) (net 12))
-  (segment (start 131.45 50.8358) (end 131.45 50.424) (width 0.5) (layer B.Cu) (net 12))
+  (segment (start 131.45 47.424) (end 127.09641 43.07041) (width 0.5) (layer F.Cu) (net 12))
   (segment (start 127.4572 54.8286) (end 131.45 50.8358) (width 0.5) (layer B.Cu) (net 12) (status 10))
+  (segment (start 131.45 50.8358) (end 131.45 50.424) (width 0.5) (layer B.Cu) (net 12))
   (segment (start 131.45 50.424) (end 131.45 47.424) (width 0.5) (layer F.Cu) (net 12))
-  (segment (start 131.45 47.424) (end 127.09641 43.07041) (width 0.5) (layer F.Cu) (net 12))
   (segment (start 98.6978 61.5) (end 101.6 58.5978) (width 0.3) (layer B.Cu) (net 13) (status 20))
   (segment (start 94.6 61.5) (end 98.6978 61.5) (width 0.3) (layer B.Cu) (net 13) (status 10))
