File: pcb/pin-check.kicad_pcb (KiCad board)
At the start: 2 copper layers, 76.2 x 52.3 mm, 55 parts, among them J1 AVR-ISP-6, J2 SJ-43514, P1 USB_C_Receptacle_USB2.0, SW1 MX-NoLED, SW2 MX-NoLED, SW3 MX-NoLED, SW4 MX-NoLED, SW7 Reset, SW8 Boot, U1 ATmega328P-PU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

Commit message: stray tracks
Routing:
- net Net-(P1-PadB5): track 56.4 -> 39.1 mm

Commit message: some changes
Parts:
- moved F1 48.9 mm to (162.2, 88.7)
- moved H7 48.1 mm to (165.1, 115.1)
- moved D1 48.1 mm to (112.1, 109.3)
- moved D3 48.1 mm to (148.9, 109.3)
- moved G*** 48.1 mm to (113.3, 77.2)
- moved H1 48.1 mm to (112.6, 115.1)
- moved H10 48.1 mm to (154.3, 115.1)
- moved H11 48.1 mm to (150.7, 115.1)
- moved H14 48.1 mm to (139.9, 115.1)
- moved H2 48.1 mm to (129.8, 97.6)
- moved H3 48.1 mm to (148.9, 97.6)
- moved H4 48.1 mm to (167.9, 97.6)
- moved J1 48.1 mm to (121.8, 73.3)
- moved P1 48.1 mm to (148.9, 66.9)
- moved R5 48.1 mm to (175.3, 78.7)
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Routing:
- net +5V: track 121.9 -> 127.3 mm
- net Net-(F1-Pad2): track 26.1 -> 27.1 mm
Other:
- board text added: "ColA"
- board text added: "ColB"
- board text added: "ColC"
- board text added: "ColD"
- board text added: "SW1"
- board text added: "SW2"
- board text added: "SW3"
- board text added: "SW4"

Commit message: also probably not
Parts:
- added U2: MCP23008-xP, Package_DIP:DIP-18_W7.62mm, B.Cu at (86.2, 79.6)

Commit message: updates
Parts:
- removed U2: MCP23008-xP, Package_DIP:DIP-18_W7.62mm
- added H18: Pad, Connector_Wire:SolderWire-0.5sqmm_1x01_D0.9mm_OD2.1mm, B.Cu at (134.0, 94.3)
- added H19: Pad, Connector_Wire:SolderWire-0.5sqmm_1x01_D0.9mm_OD2.1mm, B.Cu at (137.6, 94.3)
- added H20: Pad, Connector_Wire:SolderWire-0.5sqmm_1x01_D0.9mm_OD2.1mm, B.Cu at (141.2, 94.3)
- added H21: Pad, Connector_Wire:SolderWire-0.5sqmm_1x01_D0.9mm_OD2.1mm, B.Cu at (144.8, 94.3)
- moved J2 4.34 mm to (160.1, 68.6)
- moved J1 0.51 mm to (121.8, 72.7)
- moved R1 0.51 mm to (175.3, 89.0)
- moved R2 0.51 mm to (172.9, 88.2)
- moved R3 0.51 mm to (170.5, 87.5)
- moved R4 0.51 mm to (168.1, 86.7)
- moved C5 0.25 mm to (132.8, 87.7)
- renumbered H18 to H22, H19 to H23, H20 to H24, H21 to H25
Connections:
- J2 pad 2: /C5 -> /SCL
- J2 pad 3: /C4 -> /SDA
- R7 pad 2: /C5 -> /SCL
- R8 pad 2: /C4 -> /SDA
- U1 pad 27: /C4 -> /SDA
- U1 pad 28: /C5 -> /SCL
Routing:
- net /C5: track 63.7 -> 0.00 mm, vias 1 -> 0
- net /C4: track 62.8 -> 0.21 mm, vias 2 -> 0
- net Net-(P1-PadB5): track 39.1 -> 0.00 mm, vias 3 -> 0
- net /D-: track 40.6 -> 8.10 mm
- net /SCL: track 0.00 -> 30.8 mm
- net Net-(P1-PadA5): track 30.6 -> 0.28 mm, vias 2 -> 0
- net /SDA: track 0.00 -> 23.0 mm
- net Net-(D7-Pad1): track 43.5 -> 20.9 mm, vias 2 -> 0
- net /ColA: track 55.3 -> 57.7 mm
- net /ColD: track 62.6 -> 64.4 mm, vias 0 -> 1
- net /Reset: track 69.8 -> 71.4 mm, vias 0 -> 1
- net +5V: track 127.3 -> 126.1 mm
- net /ColC: track 36.9 -> 38.0 mm, vias 0 -> 1
- net Net-(D8-Pad1): track 34.0 -> 35.0 mm
- net /Boot: track 73.3 -> 74.2 mm, vias 0 -> 2
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Other:
- board text added: "GND"
- board text added: "I2C"
- board text added: "SCL"
- board text added: "SDA"
- board text added: "VCC"

Commit message: resolve some issues and update images
Parts:
- moved R1 23.3 mm to (156.3, 75.7), turned to 270 degrees
- moved R2 18.4 mm to (158.8, 76.4), turned to 270 degrees
- moved R6 17.2 mm to (169.0, 87.1), turned to 90 degrees
- moved F1 14.2 mm to (167.4, 75.5), turned to 90 degrees
- moved R3 13.8 mm to (161.3, 77.2), turned to 270 degrees
- moved R4 9.71 mm to (163.9, 78.0), turned to 270 degrees
- moved R5 8.89 mm to (166.4, 78.7), turned to 270 degrees
- moved R8 7.56 mm to (174.0, 81.1), turned to 270 degrees
- moved R7 3.21 mm to (171.5, 80.2), turned to 270 degrees
- moved J1 0.52 mm to (122.0, 72.2)
- moved D8 0.31 mm to (174.0, 66.1)
- moved D7 0.31 mm to (181.6, 66.1)
Routing:
- net Net-(D7-Pad1): track 20.9 -> 61.9 mm
- net Net-(D8-Pad1): track 35.0 -> 68.3 mm, vias 0 -> 1
- net /SDA: track 23.0 -> 54.9 mm, vias 0 -> 1
- net /SCL: track 30.8 -> 62.1 mm
- net /D-: track 8.10 -> 27.2 mm, vias 1 -> 0
- net Net-(P1-PadB5): track 0.00 -> 17.5 mm
- net Net-(P1-PadA5): track 0.28 -> 14.5 mm
- net /Reset: track 71.4 -> 79.4 mm, vias 1 -> 0
- net /D+: track 33.6 -> 28.0 mm, vias 2 -> 0
- net GND: track 17.3 -> 20.9 mm
- net +5V: track 126.1 -> 128.4 mm
- net Net-(F1-Pad2): track 27.1 -> 28.5 mm
- net /B3: track 55.9 -> 56.4 mm
- net /B4: track 61.6 -> 62.2 mm
- net /Boot: track 74.2 -> 73.7 mm, vias 2 -> 0

Commit message: move everything down
Parts:
- moved D1 1.00 mm to (112.1, 110.3)
- moved D2 1.00 mm to (129.8, 110.3)
- moved D3 1.00 mm to (148.9, 110.3)
- moved D4 1.00 mm to (167.9, 110.3)
- moved H1 1.00 mm to (112.6, 116.1)
- moved H10 1.00 mm to (154.3, 116.1)
- moved H11 1.00 mm to (150.7, 116.1)
- moved H12 1.00 mm to (147.1, 116.1)
- moved H13 1.00 mm to (143.5, 116.1)
- moved H14 1.00 mm to (139.9, 116.1)
- moved H15 1.00 mm to (136.3, 116.1)
- moved H16 1.00 mm to (132.7, 116.1)
- moved H17 1.00 mm to (129.1, 116.1)
- moved H18 1.00 mm to (134.0, 95.3)
- moved H19 1.00 mm to (137.6, 95.3)
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Routing:
- net Net-(D8-Pad1): track 68.3 -> 63.4 mm, vias 1 -> 2
- net /ColB: track 25.7 -> 27.1 mm
- net /D6: track 70.9 -> 72.3 mm
- net /D4: track 54.4 -> 55.7 mm
- net /C3: track 31.8 -> 33.1 mm
- net /ColA: track 58.1 -> 56.8 mm
- net /Row0: track 96.2 -> 97.5 mm
- net /D7: track 73.6 -> 74.8 mm
- net /B4: track 62.2 -> 63.2 mm
- net /B3: track 56.4 -> 57.4 mm
- net /B1: track 34.9 -> 35.9 mm
- net /SCL: track 62.1 -> 63.1 mm
- net /D1: track 48.2 -> 49.2 mm
- net /D0: track 48.9 -> 49.9 mm
- net /ColD: track 64.4 -> 65.4 mm
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Other:
- board size 76.2 x 52.3 mm -> 76.2 x 53.3 mm
